Commit message: Parametrized quadrotor simple controller urdf

File: simulation/hector_quadrotor_gazebo_plugins/urdf/quadrotor_simple_controller.urdf.xacro (robot description, xacro)
@@ -5,11 +5,11 @@
 >
   <!-- Quadrotor Simple Controller Plugin -->
-  <xacro:macro name="hector_quadrotor_simple_controller" params="model_name state_topic imu_topic">
+  <xacro:macro name="hector_quadrotor_simple_controller" params="model_name base_link state_topic imu_topic command_topic update_rate">
     <gazebo>
       <plugin name="hector_quadrotor_simple_controller" filename="libhector_quadrotor_gazebo_simple_controller.so">
         <alwaysOn>true</alwaysOn>
-        <updateRate>0.0</updateRate>
-        <bodyName>base_link</bodyName>
-        <topicName>${model_name}/cmd_vel</topicName>
+        <updateRate>${update_rate}</updateRate>
+        <bodyName>${base_link}</bodyName>
+        <topicName>${model_name}/${command_topic}</topicName>
         <stateTopic>${model_name}/${state_topic}</stateTopic>
         <imuTopic>${model_name}/${imu_topic}</imuTopic>

Commit message: Update rate was deprecated. Removed it from simple controller urdf macro

File: simulation/hector_quadrotor_gazebo_plugins/urdf/quadrotor_simple_controller.urdf.xacro (robot description, xacro)
@@ -5,9 +5,8 @@
 >
   <!-- Quadrotor Simple Controller Plugin -->
-  <xacro:macro name="hector_quadrotor_simple_controller" params="model_name base_link state_topic imu_topic command_topic update_rate">
+  <xacro:macro name="hector_quadrotor_simple_controller" params="model_name base_link state_topic imu_topic command_topic">
     <gazebo>
       <plugin name="hector_quadrotor_simple_controller" filename="libhector_quadrotor_gazebo_simple_controller.so">
         <alwaysOn>true</alwaysOn>
-        <updateRate>${update_rate}</updateRate>
         <bodyName>${base_link}</bodyName>
         <topicName>${model_name}/${command_topic}</topicName>
