Commit message: Parametrized other urdf files in hector package

File: simulation/hector_quadrotor_gazebo_plugins/urdf/quadrotor_plugins.urdf.xacro (robot description, xacro)
@@ -8,8 +8,9 @@
   <xacro:include filename="$(find hector_quadrotor_gazebo_plugins)/urdf/quadrotor_controller.urdf.xacro" /-->
   <!-- Quadrotor Gazebo Plugins -->
-  <xacro:macro name="quadrotor_plugins" params="model_name">
+  <xacro:macro name="quadrotor_plugins" params="model_name base_link">
     <canonicalBody>base_link</canonicalBody>
-    <xacro:quadrotor_sensors model_name="${model_name}"/>
-    <xacro:quadrotor_simple_controller model_name="${model_name}"  state_topic="ground_truth/state" imu_topic="raw_imu"/>
+    <xacro:quadrotor_sensors model_name="${model_name}" base_link="${base_link}"/>
+    <xacro:quadrotor_simple_controller model_name="${model_name}"  state_topic="ground_truth/state" imu_topic="raw_imu"
+      base_link="${base_link}" command_topic="cmd_vel"/>
   </xacro:macro>
 </robot>

File: simulation/hector_quadrotor_gazebo_plugins/urdf/quadrotor_sensors.urdf.xacro (robot description, xacro)
@@ -6,9 +6,9 @@
 >
   <!-- Quadrotor Sensor Plugins -->
-  <xacro:macro name="quadrotor_sensors" params="model_name">
+  <xacro:macro name="quadrotor_sensors" params="model_name base_link">
     <gazebo>
       <plugin name="quadrotor_imu_sim" filename="libhector_gazebo_ros_imu.so">
         <updateRate>100.0</updateRate>
-        <bodyName>base_link</bodyName>
+        <bodyName>${base_link}</bodyName>
         <topicName>${model_name}/raw_imu</topicName>
         <rpyOffsets>0 0 0</rpyOffsets> <!-- deprecated -->
@@ -23,5 +23,5 @@
       <plugin name="quadrotor_baro_sim" filename="libhector_gazebo_ros_baro.so">
         <updateRate>10.0</updateRate>
-        <bodyName>base_link</bodyName>
+        <bodyName>${base_link}</bodyName>
         <topicName>${model_name}/pressure_height</topicName>
         <altimeterTopicName>${model_name}/altimeter</altimeterTopicName>
@@ -32,5 +32,5 @@
       <plugin name="quadrotor_magnetic_sim" filename="libhector_gazebo_ros_magnetic.so">
         <updateRate>10.0</updateRate>
-        <bodyName>base_link</bodyName>
+        <bodyName>${base_link}</bodyName>
         <topicName>${model_name}/magnetic</topicName>
         <offset>0 0 0</offset>
@@ -40,5 +40,5 @@
       <plugin name="quadrotor_gps_sim" filename="libhector_gazebo_ros_gps.so">
         <updateRate>4.0</updateRate>
-        <bodyName>base_link</bodyName>
+        <bodyName>${base_link}</bodyName>
         <topicName>${model_name}/fix</topicName>
         <velocityTopicName>${model_name}/fix_velocity</velocityTopicName>
@@ -50,5 +50,5 @@
       <plugin name="quadrotor_groundtruth_sim" filename="libgazebo_ros_p3d.so">
         <updateRate>100.0</updateRate>
-        <bodyName>base_link</bodyName>
+        <bodyName>${base_link}</bodyName>
         <topicName>${model_name}/ground_truth/state</topicName>
         <gaussianNoise>0.0</gaussianNoise>
