Commit message: Spawn a simple quad

File: hal/urdf/grvc_quadrotor_base.urdf.xacro (robot description, xacro)
@@ -33,5 +33,5 @@
         <origin xyz="0.0 0.0 0.0" rpy="0.0 0.0 0.0" />
         <geometry>
-          <mesh filename="package://grvc_quadrotor_hal/models/propellers.dae"/>
+          <mesh filename="package://grvc_quadrotor_hal/model/propellers.dae"/>
         </geometry>
       </visual>
@@ -61,5 +61,5 @@
         <origin xyz="0 0 -0.25" rpy="0 0 0" />
         <geometry>
-          <mesh filename="package://grvc_quadrotor_hal/models/grvc_quad.dae"/>
+          <mesh filename="package://grvc_quadrotor_hal/model/grvc_quad.dae"/>
         </geometry>
       </visual>
@@ -67,5 +67,5 @@
         <origin xyz="0 0 -0.25" rpy="0 0 0" />
         <geometry>
-          <mesh filename="package://grvc_quadrotor_hal/models/grvc_quad_simplified.stl"/>
+          <mesh filename="package://grvc_quadrotor_hal/model/grvc_quad_simplified.stl"/>
         </geometry>
       </collision>
