Commit message: Launch the right simulation plugin in gazebo

File: hal/urdf/grvc_quadrotor.urdf.xacro (robot description, xacro)
@@ -9,9 +9,8 @@
 <robot name="grvc_quadrotor" xmlns:xacro="http://ros.org/wiki/xacro">
   <xacro:property name="M_PI" value="3.1415926535897931" />
-  <xacro:property name="id" value="1" />
   <!-- Included URDF Files -->
   <xacro:include filename="$(find grvc_quadrotor_hal)/urdf/grvc_quadrotor_base.urdf.xacro" />
   <!-- Instantiate quadrotor_base_macro once (has no parameters atm) -->
   <!-- model_name must be ual_${id} for ual node to find the uav -->
-  <xacro:quadrotor_base_macro id="${id}" model_name="uav_${id}"/>
+  <xacro:quadrotor_base_macro id="1" model_name="grvc_hal"/>
 </robot>

File: hal/urdf/grvc_quadrotor_base.urdf.xacro (robot description, xacro)
@@ -11,5 +11,5 @@
 xmlns:interface="http://playerstage.sourceforge.net/gazebo/xmlschema/#interface"
 xmlns:xacro="http://ros.org/wiki/xacro">
-  <xacro:include filename="$(find hector_quadrotor_gazebo_plugins)/urdf/quadrotor_plugins.urdf.xacro" />
+  <xacro:include filename="$(find grvc_quadrotor_gazebo)/urdf/quadrotor_plugins.urdf.xacro" />
   <property name="pi" value="3.1415926535897931" />
   <property name="col_box_l1" value="0.05" />
@@ -79,6 +79,5 @@
     </gazebo>
     <!-- Gazebo Plugins -->
-    <xacro:multi_quadrotor_plugins model_name="${model_name}" base_link="base_link_${id}"/>
-    <!--xacro:multi_bonebraker_arm_controller base_link="base_link_${id}" robot_id ="${id}" /-->
+    <xacro:quadrotor_plugins model_name="${model_name}" base_link="base_link_${id}"/>
   </xacro:macro>
 </robot>

File: simulation/grvc_quadrotor_gazebo/urdf/quadrotor_plugins.urdf.xacro (robot description, xacro)
@@ -1,6 +1,6 @@
 <?xml version="1.0"?>
 <robot xmlns:xacro="http://ros.org/wiki/xacro">
-  <xacro:include filename="$(find hector_quadrotor_gazebo_plugins)/urdf/quadrotor_sensors.urdf.xacro" />
-  <xacro:include filename="$(find hector_quadrotor_gazebo_plugins)/urdf/quadrotor_simple_controller.urdf.xacro" />
+  <xacro:include filename="$(find grvc_quadrotor_gazebo)/urdf/quadrotor_sensors.urdf.xacro" />
+  <xacro:include filename="$(find grvc_quadrotor_gazebo)/urdf/quadrotor_simple_controller.urdf.xacro" />
   <!-- Quadrotor Gazebo Plugins -->
   <xacro:macro name="quadrotor_plugins" params="model_name base_link">

File: simulation/grvc_quadrotor_gazebo/urdf/quadrotor_simple_controller.urdf.xacro (robot description, xacro)
@@ -5,7 +5,7 @@
 >
   <!-- Quadrotor Simple Controller Plugin -->
-  <xacro:macro name="hector_quadrotor_simple_controller" params="model_name base_link state_topic imu_topic command_topic">
+  <xacro:macro name="quadrotor_simple_controller" params="model_name base_link state_topic imu_topic command_topic">
     <gazebo>
-      <plugin name="hector_quadrotor_simple_controller" filename="libhector_quadrotor_gazebo_simple_controller.so">
+      <plugin name="grvc_quadrotor_gazebo_plugin" filename="libgrvc_quadrotor_gazebo.so">
         <alwaysOn>true</alwaysOn>
         <bodyName>${base_link}</bodyName>
