Commit message: Support launching multiple quadrotors

File: simulation/grvc_quadrotor_gazebo/urdf/grvc_quadrotor.urdf.xacro (robot description, xacro)
@@ -9,8 +9,10 @@
 <robot name="grvc_quadrotor" xmlns:xacro="http://ros.org/wiki/xacro">
   <xacro:property name="M_PI" value="3.1415926535897931" />
+  <xacro:arg name="model_name" default="grvc_gazebo"/>
+  <xacro:arg name="id" default="1"/>
   <!-- Included URDF Files -->
-  <xacro:include filename="$(find grvc_quadrotor_hal)/urdf/grvc_quadrotor_base.urdf.xacro" />
+  <xacro:include filename="$(find grvc_quadrotor_gazebo)/urdf/grvc_quadrotor_base.urdf.xacro" />
   <!-- Instantiate quadrotor_base_macro once (has no parameters atm) -->
   <!-- model_name must be ual_${id} for ual node to find the uav -->
-  <xacro:quadrotor_base_macro id="1" model_name="grvc_hal_gazebo"/>
+  <xacro:quadrotor_base_macro id="$(arg id)" model_name="$(arg model_name)"/>
 </robot>

File: simulation/grvc_quadrotor_gazebo/urdf/grvc_quadrotor_base.urdf.xacro (robot description, xacro)
@@ -33,5 +33,5 @@
         <origin xyz="0.0 0.0 0.0" rpy="0.0 0.0 0.0" />
         <geometry>
-          <mesh filename="package://grvc_quadrotor_hal/model/propellers.dae"/>
+          <mesh filename="package://grvc_quadrotor_gazebo/model/propellers.dae"/>
         </geometry>
       </visual>
@@ -61,5 +61,5 @@
         <origin xyz="0 0 -0.25" rpy="0 0 0" />
         <geometry>
-          <mesh filename="package://grvc_quadrotor_hal/model/grvc_quad.dae"/>
+          <mesh filename="package://grvc_quadrotor_gazebo/model/grvc_quad.dae"/>
         </geometry>
       </visual>
@@ -67,5 +67,5 @@
         <origin xyz="0 0 -0.25" rpy="0 0 0" />
         <geometry>
-          <mesh filename="package://grvc_quadrotor_hal/model/grvc_quad_simplified.stl"/>
+          <mesh filename="package://grvc_quadrotor_gazebo/model/grvc_quad_simplified.stl"/>
         </geometry>
       </collision>
